Commit message: multiple sensors added

File: models/rotors_description/urdf_old/component_snippets.xacro (robot description, xacro)
@@ -17,6 +17,4 @@
 -->
 <robot xmlns:xacro="http://ros.org/wiki/xacro">
-	<xacro:property name="DEG2RAD" value="0.017453292519943295"/>
-  <xacro:property name="M_PI" value="3.1415926535897931" />
   <!-- Macro to add logging to a bag file. -->
   <xacro:macro name="bag_plugin_macro"
@@ -129,65 +127,4 @@
     </gazebo>
   </xacro:macro>
-    <!-- Macro to add the range_plugin. FIll here! -->
-	<xacro:macro name="sonar_sensor" params="name parent *origin ros_topic update_rate min_range max_range field_of_view ray_count">
-    <joint name="${name}_joint" type="fixed">
-      <xacro:insert_block name="origin" />
-      <parent link="${parent}"/>
-      <child link="${name}_link"/>
-    </joint>
-    <link name="${name}_link">
-      <inertial>
-        <mass value="0.001" />
-        <origin xyz="0 0 0" rpy="0 0 0" />
-        <inertia ixx="0.000000017" ixy="0" ixz="0" iyy="0.000000017" iyz="0" izz="0.000000017" />
-      </inertial>
-      <visual>
-        <origin xyz="0 0 0" rpy="0 0 0" />
-        <geometry>
-          <box size="0.01 0.01 0.01" />
-        </geometry>
-      </visual>
-      <collision>
-        <origin xyz="0 0 0" rpy="0 0 0" />
-        <geometry>
-          <box size="0.01 0.01 0.01" />
-        </geometry>
-      </collision>
-    </link>
-    <gazebo reference="${name}_link">
-      <sensor type="ray" name="${name}">
-        <always_on>true</always_on>
-        <update_rate>${update_rate}</update_rate>
-        <pose>0 0 0 0 0 0</pose>
-        <visualize>false</visualize>
-        <ray>
-          <scan>
-            <horizontal>
-              <samples>${ray_count}</samples>
-              <resolution>1</resolution>
-              <min_angle>-${field_of_view/2}</min_angle>
-              <max_angle> ${field_of_view/2}</max_angle>
-            </horizontal>
-            <vertical>
-              <samples>${ray_count}</samples>
-              <resolution>1</resolution>
-              <min_angle>-${field_of_view/2}</min_angle>
-              <max_angle> ${field_of_view/2}</max_angle>
-            </vertical>
-          </scan>
-          <range>
-            <min>${min_range}</min>
-            <max>${max_range}</max>
-            <resolution>0.01</resolution>
-          </range>
-        </ray>
-        <plugin name="gazebo_ros_${name}_controller" filename="libhector_gazebo_ros_sonar.so">
-          <gaussianNoise>0.005</gaussianNoise>
-          <topicName>${ros_topic}</topicName>
-          <frameId>${name}_link</frameId>
-        </plugin>
-      </sensor>
-    </gazebo>
-  </xacro:macro>
   <!-- Macro to add the mavlink interface. -->
   <xacro:macro name="mavlink_interface_macro" params="namespace imu_sub_topic gps_sub_topic mavlink_addr mavlink_udp_port serial_enabled serial_device baudrate qgc_addr qgc_udp_port hil_mode hil_state_level vehicle_is_tailsitter send_odometry">
@@ -422,94 +359,4 @@
         <windGustForceMean>${wind_gust_force_mean}</windGustForceMean> <!-- [N] -->
       </plugin>
-    </gazebo>
-  </xacro:macro>
-  <!-- VI sensor macros -->
-  <!-- Macro to add a VI-sensor camera. -->
-  <xacro:macro name="vi_sensor_camera_macro"
-    params="namespace parent_link camera_suffix frame_rate *origin">
-    <xacro:camera_macro
-      namespace="${namespace}"
-      parent_link="${parent_link}"
-      camera_suffix="${camera_suffix}"
-      frame_rate="${frame_rate}"
-      horizontal_fov="1.3962634"
-      image_width="752"
-      image_height="480"
-      image_format="L8"
-      min_distance="0.02"
-      max_distance="30"
-      noise_mean="0.0"
-      noise_stddev="0.007"
-      enable_visual="false">
-      <cylinder length="0.01" radius="0.007" />
-      <xacro:insert_block name="origin" />
-    </xacro:camera_macro>
-  </xacro:macro>
-  <!-- Macro to add a depth camera on the VI-sensor. -->
-  <xacro:macro name="vi_sensor_depth_macro"
-    params="namespace parent_link camera_suffix frame_rate *origin">
-    <link name="${namespace}/camera_${camera_suffix}_link">
-      <collision>
-        <origin xyz="0 0 0" rpy="0 0 0" />
-        <geometry>
-          <cylinder length="0.01" radius="0.007" />
-        </geometry>
-      </collision>
-      <inertial>
-        <mass value="1e-5" />
-        <origin xyz="0 0 0" rpy="0 0 0" />
-        <inertia ixx="1e-6" ixy="0" ixz="0" iyy="1e-6" iyz="0" izz="1e-6" />
-      </inertial>
-    </link>
-    <joint name="${namespace}/camera_${camera_suffix}_joint" type="fixed">
-      <xacro:insert_block name="origin" />
-      <parent link="${parent_link}" />
-      <child link="${namespace}/camera_${camera_suffix}_link" />
-      <limit upper="0" lower="0" effort="0" velocity="0" />
-    </joint>
-    <!-- Optical center of camera -->
-    <link name="${namespace}/camera_${camera_suffix}_optical_center_link" />
-    <joint name="${namespace}/camera_${camera_suffix}_optical_center_joint" type="fixed">
-      <origin xyz="0 0 0" rpy="${-3.1415/2} 0 ${-3.1415/2}" />
-      <parent link="${namespace}/camera_${camera_suffix}_link" />
-      <child link="${namespace}/camera_${camera_suffix}_optical_center_link" />
-      <limit upper="0" lower="0" effort="0" velocity="0" />
-    </joint>
-    <gazebo reference="${namespace}/camera_${camera_suffix}_link">
-      <sensor type="depth" name="${namespace}_camera_{camera_suffix}">
-        <always_on>true</always_on>
-        <update_rate>${frame_rate}</update_rate>
-        <camera>
-          <horizontal_fov>2</horizontal_fov>
-          <image>
-            <format>L8</format>
-            <width>640</width>
-            <height>480</height>
-          </image>
-          <clip>
-            <near>0.01</near>
-            <far>100</far>
-          </clip>
-        </camera>
-        <plugin name="${namespace}_camera_{camera_suffix}" filename="libgazebo_ros_openni_kinect.so">
-          <robotNamespace>${namespace}</robotNamespace>
-          <alwaysOn>true</alwaysOn>
-          <baseline>0.11</baseline>
-          <updateRate>${frame_rate}</updateRate>
-          <cameraName>camera_${camera_suffix}</cameraName>
-          <imageTopicName>camera/image_raw</imageTopicName>
-          <cameraInfoTopicName>camera/camera_info</cameraInfoTopicName>
-          <depthImageTopicName>depth/disparity</depthImageTopicName>
-          <depthImageCameraInfoTopicName>depth/camera_info</depthImageCameraInfoTopicName>
-          <pointCloudTopicName>depth/points</pointCloudTopicName>
-          <frameName>camera_${camera_suffix}_optical_center_link</frameName>
-          <pointCloudCutoff>0.5</pointCloudCutoff>
-          <distortionK1>0.0</distortionK1>
-          <distortionK2>0.0</distortionK2>
-          <distortionK3>0.0</distortionK3>
-          <distortionT1>0.0</distortionT1>
-          <distortionT2>0.0</distortionT2>
-        </plugin>
-      </sensor>
     </gazebo>
   </xacro:macro>
@@ -705,205 +552,3 @@
     </xacro:imu_plugin_macro>
   </xacro:macro>
-	<xacro:macro name="hokuyo_utm30lx_model" params="name parent *origin">
-    <joint name="${name}_joint" type="fixed">
-      <xacro:insert_block name="origin" />
-      <parent link="${parent}"/>
-      <child link="${name}_frame"/>
-    </joint>
-    <link name="${name}_frame">
-      <inertial>
-        <mass value="0.270" />
-        <origin xyz="0 0 0" rpy="0 0 0" />
-        <inertia ixx="2.632e-4" ixy="0" ixz="0" iyy="2.632e-4" iyz="0" izz="1.62e-4" />
-      </inertial>
-      <visual>
-        <origin xyz="0 0 0" rpy="0 0 0" />
-        <geometry>
-        <box size="0.025 0.025 0.035" />
-        </geometry>
-      </visual>
-      <collision>
-        <origin xyz="0 0 0" rpy="0 0 0" />
-        <geometry>
-        <box size="0.025 0.025 0.035" />
-      </geometry>
-      </collision>
-    </link>
-  </xacro:macro>
-	<xacro:macro name="hokuyo_utm30lx" params="name parent *origin ros_topic update_rate ray_count min_angle max_angle">
-      <xacro:hokuyo_utm30lx_model name="${name}" parent="${parent}">
-        <xacro:insert_block name="origin" />
-      </xacro:hokuyo_utm30lx_model>
-      <gazebo reference="${name}_frame">
-        <sensor type="ray" name="${name}">
-          <always_on>true</always_on>
-          <update_rate>${update_rate}</update_rate>
-          <pose>0 0 0.0 0 0 0</pose>
-          <visualize>false</visualize>
-          <ray>
-            <scan>
-              <horizontal>
-                <samples>${ray_count}</samples>
-                <resolution>1</resolution>
-                <min_angle>${min_angle * M_PI/180}</min_angle>
-                <max_angle>${max_angle * M_PI/180}</max_angle>
-              </horizontal>
-            </scan>
-            <range>
-              <min>0.2</min>
-              <max>30.0</max>
-              <resolution>0.01</resolution>
-            </range>
-            <noise>
-              <type>gaussian</type>
-              <mean>0.0</mean>
-              <stddev>0.004</stddev>
-            </noise>
-          </ray>
-          <plugin name="gazebo_ros_${name}_controller" filename="libgazebo_ros_laser.so">
-            <topicName>${ros_topic}</topicName>
-            <frameName>${name}_frame</frameName>
-          </plugin>
-        </sensor>
-      </gazebo>
-   </xacro:macro>
-  <xacro:macro name="xtion_pro_live_rgbd_camera_gazebo" params="name">
-    <gazebo reference="${name}">
-      <!-- Depth (IR) -->
-      <sensor type="depth" name="${name}_frame_sensor">
-        <always_on>true</always_on>
-        <update_rate>6.0</update_rate>
-        <camera>
-          <horizontal_fov>${100.0 * DEG2RAD}</horizontal_fov>
-          <image>
-           <format>R8G8B8</format>
-            <width>1360</width>
-						<height>768</height>
-          </image>
-          <clip>
-            <near>0.2</near>
-            <far>6.0</far>
-          </clip>
-        </camera>
-        <plugin name="${name}_frame_controller" filename="libgazebo_ros_openni_kinect.so">
-          <alwaysOn>true</alwaysOn>
-          <updateRate>5.0</updateRate>
-          <cameraName>${name}</cameraName>
-          <imageTopicName>ir/image_raw</imageTopicName>
-          <cameraInfoTopicName>ir/camera_info</cameraInfoTopicName>
-          <depthImageTopicName>depth/image_raw</depthImageTopicName>
-          <depthImageCameraInfoTopicName>depth/camera_info</depthImageCameraInfoTopicName>
-          <pointCloudTopicName>depth/points</pointCloudTopicName>
-          <frameName>${name}_optical_frame</frameName>
-          <pointCloudCutoff>0.05</pointCloudCutoff>
-          <pointCloudCutoffMax>5</pointCloudCutoffMax>
-          <rangeMax>0.5</rangeMax>
-          <!-- Distortion parameters not supported in gazebo 1.9.* plugins -->
-          <!--distortionK1>0.00000001</distortionK1>
-          <distortionK2>0.00000001</distortionK2>
-          <distortionK3>0.00000001</distortionK3>
-          <distortionT1>0.00000001</distortionT1>
-          <distortionT2>0.00000001</distortionT2-->
-        </plugin>
-      </sensor>
-      <!-- RGB -->
-      <sensor type="depth" name="${name}_frame_sensor">
-        <always_on>true</always_on>
-        <update_rate>6.0</update_rate>
-        <camera>
-          <horizontal_fov>${100.0 * DEG2RAD}</horizontal_fov>
-          <image>
-            <format>R8G8B8</format>
-            <width>1360</width>
-            <height>768</height>
-          </image>
-          <clip>
-            <near>0.2</near>
-            <far>6.0</far>
-          </clip>
-        </camera>
-        <plugin name="${name}_frame_controller" filename="libgazebo_ros_openni_kinect.so">
-          <alwaysOn>true</alwaysOn>
-          <updateRate>6.0</updateRate>
-          <cameraName>${name}</cameraName>
-          <imageTopicName>rgb/image_raw</imageTopicName>
-          <cameraInfoTopicName>rgb/camera_info</cameraInfoTopicName>
-          <pointCloudTopicName>rgb/points</pointCloudTopicName>
-          <depthImageTopicName>depth/image_raw</depthImageTopicName>
-          <depthImageCameraInfoTopicName>depth/camera_info</depthImageCameraInfoTopicName>
-          <frameName>${name}_optical_frame</frameName>
-          <pointCloudCutoff>0.05</pointCloudCutoff>
-          <pointCloudCutoffMax>5</pointCloudCutoffMax>
-          <rangeMax>2.5</rangeMax>
-        </plugin>
-     </sensor>
-    </gazebo>
-  </xacro:macro>
- <xacro:macro name="xtion_pro_live" params="name parent *origin *optical_origin">
-    <!-- frames in the center of the camera -->
-    <joint name="${name}_joint" type="fixed">
-      <xacro:insert_block name="origin"/>
-      <parent link="${parent}"/>
-      <child link="${name}"/>
-    </joint>
-    <link name="${name}">
-      <inertial>
-        <origin xyz="-0.00936000000 -0.00003000000 -0.00273000000" rpy="0 0 0"/>
-        <mass value="0.21970000000"/>
-        <inertia ixx="0.00000429247" ixy="0.00000000000" ixz="0.00000002565"
-                 iyy="0.00000008027" iyz="0.00000000000"
-                 izz="0.00000427339"/>
-      </inertial>
-      <visual>
-        <origin xyz="0 0 0" rpy="0 0 0"/>
-        <geometry>
-          <box size="0.01 0.08 0.01" />
-        </geometry>
-        <material name="DarkGrey"/>
-      </visual>
-    </link>
-    <joint name="${name}_optical_joint" type="fixed">
-      <xacro:insert_block name="optical_origin"/>
-      <parent link="${name}"/>
-      <child link="${name}_optical_frame"/>
-    </joint>
-    <link name="${name}_optical_frame">
-      <dummy_inertial/>
-    </link>
-    <!-- Depth sensor frames -->
-    <joint name="${name}_depth_joint" type="fixed">
-      <origin xyz="0.0 0.049 0.0" rpy="0 0 0"/>
-      <parent link="${name}"/>
-      <child link="${name}_depth_frame"/>
-    </joint>
-    <link name="${name}_depth_frame">
-      <dummy_inertial/>
-    </link>
-    <joint name="${name}_depth_optical_joint" type="fixed">
-      <origin xyz="0 0 0" rpy="${-90.0 * DEG2RAD} 0.0 ${-90.0 * DEG2RAD}"/>
-      <parent link="${name}_depth_frame"/>
-      <child link="${name}_depth_optical_frame"/>
-    </joint>
-    <link name="${name}_depth_optical_frame">
-      <dummy_inertial/>
-    </link>
-    <!-- RGB sensor frames -->
-    <joint name="${name}_rgb_joint" type="fixed">
-      <origin xyz="0.0 0.022 0.0" rpy="0 0 0"/>
-      <parent link="${name}"/>
-      <child link="${name}_rgb_frame"/>
-    </joint>
-    <link name="${name}_rgb_frame">
-      <dummy_inertial/>
-    </link>
-    <joint name="${name}_rgb_optical_joint" type="fixed">
-      <origin xyz="0 0 0" rpy="${-90.0 * DEG2RAD} 0.0 ${-90.0 * DEG2RAD}"/>
-      <parent link="${name}_rgb_frame"/>
-      <child link="${name}_rgb_optical_frame"/>
-    </joint>
-    <link name="${name}_rgb_optical_frame">
-      <dummy_inertial/>
-    </link>
-    <xacro:xtion_pro_live_rgbd_camera_gazebo name="${name}"/>
-  </xacro:macro>
 </robot>

File: models/rotors_description/urdf_old/iris_base.xacro (robot description, xacro)
@@ -65,108 +65,4 @@
   </xacro:mavlink_interface_macro>
   </xacro:if>
-	<!-- Mount a Camera -->
-<!--
-	<xacro:camera_macro
-		  namespace="${namespace}"
-			parent_link="base_link"
-			camera_suffix="raw"
-			frame_rate="30"
-			horizontal_fov="1.4"
-			image_width="1280"
-			image_height="720"
-			image_format="B8G8R8"
-			min_distance="0.02"
-			max_distance="300"
-			noise_mean="0.0"
-			noise_stddev="0.008"
-			enable_visual="1"
-		>
-		<box size="0.02 0.02 0.02" />
-		<origin xyz="0.12 0 -0.02" rpy="0.0 1.1 0.0" />
-	</xacro:camera_macro>
--->
-	<!---->
-  <xacro:xtion_pro_live name="rgbd_camera" parent="base_link">
-	 	<origin xyz="0.11 0.0 -0.02" rpy="0.0 0.95 0.0"/>
-    <origin xyz="0 0 0" rpy="0.0 0 0.0"/>
-	</xacro:xtion_pro_live>
-	    <xacro:hokuyo_utm30lx name="laser_scanner" parent="base_link" ros_topic="scan" update_rate="40" ray_count="1081" min_angle="-135" max_angle="135">
-      <origin xyz="0.0 0.0 0.06" rpy="${M_PI} 0 0"/>
-    </xacro:hokuyo_utm30lx>
-	<xacro:macro name="hokuyo_utm30lx_model" params="name parent *origin">
-    <joint name="${name}_joint" type="fixed">
-      <xacro:insert_block name="origin" />
-      <parent link="${parent}"/>
-      <child link="${name}_frame"/>
-    </joint>
-    <link name="${name}_frame">
-      <inertial>
-        <mass value="0.270" />
-        <origin xyz="0 0 0" rpy="0 0 0" />
-        <inertia ixx="2.632e-4" ixy="0" ixz="0" iyy="2.632e-4" iyz="0" izz="1.62e-4" />
-      </inertial>
-      <visual>
-        <origin xyz="0 0 0" rpy="0 0 0" />
-        <geometry>
-        <box size="0.025 0.025 0.035" />
-        </geometry>
-      </visual>
-      <collision>
-        <origin xyz="0 0 0" rpy="0 0 0" />
-        <geometry>
-        <box size="0.025 0.025 0.035" />
-      </geometry>
-      </collision>
-    </link>
-  </xacro:macro>
-	<xacro:macro name="hokuyo_utm30lx" params="name parent *origin ros_topic update_rate ray_count min_angle max_angle">
-      <xacro:hokuyo_utm30lx_model name="${name}" parent="${parent}">
-        <xacro:insert_block name="origin" />
-      </xacro:hokuyo_utm30lx_model>
-      <gazebo reference="${name}_frame">
-        <sensor type="ray" name="${name}">
-          <always_on>true</always_on>
-          <update_rate>${update_rate}</update_rate>
-          <pose>0 0 0.0 0 0 0</pose>
-          <visualize>false</visualize>
-          <ray>
-            <scan>
-              <horizontal>
-                <samples>${ray_count}</samples>
-                <resolution>1</resolution>
-                <min_angle>${min_angle * M_PI/180}</min_angle>
-                <max_angle>${max_angle * M_PI/180}</max_angle>
-              </horizontal>
-            </scan>
-            <range>
-              <min>0.2</min>
-              <max>30.0</max>
-              <resolution>0.01</resolution>
-            </range>
-            <noise>
-              <type>gaussian</type>
-              <mean>0.0</mean>
-              <stddev>0.004</stddev>
-            </noise>
-          </ray>
-          <plugin name="gazebo_ros_${name}_controller" filename="libgazebo_ros_laser.so">
-            <topicName>${ros_topic}</topicName>
-            <frameName>${name}_frame</frameName>
-          </plugin>
-        </sensor>
-      </gazebo>
-   </xacro:macro>
-	<xacro:sonar_sensor
-		name="sonar"
-		parent="base_link"
-		ros_topic="sonar"
-		min_range="0.2"
-		max_range="8.0"
-		field_of_view="10"
-		ray_count="2"
-		update_rate="5"
-	>
-  <origin xyz="0.0 0.0 -0.04" rpy="0 0 3.14" />
-	</xacro:sonar_sensor>
   <!-- Mount an ADIS16448 IMU. -->
   <xacro:imu_plugin_macro
