Commit message: removed laser scanner

File: models/rotors_description/urdf/with_sensors/iris_base_with_sensors.xacro (robot description, xacro)
@@ -89,86 +89,9 @@
     <origin xyz="0 0 0" rpy="0.0 0 0.0"/>
 	</xacro:xtion_pro_live>
+-->
+<!--
 	    <xacro:hokuyo_utm30lx name="laser_scanner" parent="base_link" ros_topic="scan" update_rate="40" ray_count="1081" min_angle="-135" max_angle="135">
-      <origin xyz="0.0 0.0 0.06" rpy="${M_PI} 0 0"/>
+      <origin xyz="0.3 0.2 0.06" rpy="${M_PI} 0 0"/>
     </xacro:hokuyo_utm30lx>
--->
-	<!--
-	<xacro:macro name="hokuyo_utm30lx_model" params="name parent *origin">
-    <joint name="${name}_joint" type="fixed">
-      <xacro:insert_block name="origin" />
-      <parent link="${parent}"/>
-      <child link="${name}_frame"/>
-    </joint>
-    <link name="${name}_frame">
-      <inertial>
-        <mass value="0.270" />
-        <origin xyz="0 0 0" rpy="0 0 0" />
-        <inertia ixx="2.632e-4" ixy="0" ixz="0" iyy="2.632e-4" iyz="0" izz="1.62e-4" />
-      </inertial>
-      <visual>
-        <origin xyz="0 0 0" rpy="0 0 0" />
-        <geometry>
-        <box size="0.025 0.025 0.035" />
-        </geometry>
-      </visual>
-      <collision>
-        <origin xyz="0 0 0" rpy="0 0 0" />
-        <geometry>
-        <box size="0.025 0.025 0.035" />
-      </geometry>
-      </collision>
-    </link>
-  </xacro:macro>
-	<xacro:macro name="hokuyo_utm30lx" params="name parent *origin ros_topic update_rate ray_count min_angle max_angle">
-      <xacro:hokuyo_utm30lx_model name="${name}" parent="${parent}">
-        <xacro:insert_block name="origin" />
-      </xacro:hokuyo_utm30lx_model>
-      <gazebo reference="${name}_frame">
-        <sensor type="ray" name="${name}">
-          <always_on>true</always_on>
-          <update_rate>${update_rate}</update_rate>
-          <pose>0 0 0.0 0 0 0</pose>
-          <visualize>false</visualize>
-          <ray>
-            <scan>
-              <horizontal>
-                <samples>${ray_count}</samples>
-                <resolution>1</resolution>
-                <min_angle>${min_angle * M_PI/180}</min_angle>
-                <max_angle>${max_angle * M_PI/180}</max_angle>
-              </horizontal>
-            </scan>
-            <range>
-              <min>0.2</min>
-              <max>30.0</max>
-              <resolution>0.01</resolution>
-            </range>
-            <noise>
-              <type>gaussian</type>
-              <mean>0.0</mean>
-              <stddev>0.004</stddev>
-            </noise>
-          </ray>
-          <plugin name="gazebo_ros_${name}_controller" filename="libgazebo_ros_laser.so">
-            <topicName>${ros_topic}</topicName>
-            <frameName>${name}_frame</frameName>
-          </plugin>
-        </sensor>
-      </gazebo>
-   </xacro:macro>
-	-->
-	<!--
-	<xacro:sonar_sensor
-		name="sonar"
-		parent="base_link"
-		ros_topic="sonar"
-		min_range="0.2"
-		max_range="8.0"
-		field_of_view="10"
-		ray_count="2"
-		update_rate="5"
-	>
-  <origin xyz="0.0 0.0 -0.04" rpy="0 0 3.14" />
-	</xacro:sonar_sensor>
 	-->
   <!-- Mount an ADIS16448 IMU. -->

Commit message: added sonar in lpe

File: models/rotors_description/urdf/with_sensors/iris_base_with_sensors.xacro (robot description, xacro)
@@ -114,4 +114,16 @@
     <origin xyz="0 0 0" rpy="0 0 0" />
   </xacro:imu_plugin_macro>
+	<xacro:sonar_sensor
+		name="sonar"
+		parent="base_link"
+		ros_topic="distance"
+		min_range="0.2"
+		max_range="8.0"
+		field_of_view="10"
+		ray_count="2"
+		update_rate="5"
+	>
+	  <origin xyz="0.0 0.0 -0.04" rpy="0 0 3.14" />
+	</xacro:sonar_sensor>
   <xacro:if value="$(arg enable_ground_truth)">
     <!-- Mount an IMU providing ground truth. -->
