Commit message: new laser position

File: models/rotors_description/urdf/with_camera/iris_base_with_camera.xacro (robot description, xacro)
@@ -91,5 +91,5 @@
 -->
   <xacro:hokuyo_utm30lx name="laser_scanner" parent="base_link" ros_topic="scan" update_rate="40" ray_count="1081" min_angle="-135" max_angle="135">
-    <origin xyz="0.3 0.2 0.06" rpy="${M_PI} 0 0"/>
+    <origin xyz="0.0 0.0 0.06" rpy="${M_PI} 0 0"/>
   </xacro:hokuyo_utm30lx>
   <!-- Mount an ADIS16448 IMU. -->
