Commit message: new terrain follower drone model and world

File: models/rotors_description/urdf/with_terrain_sensors/iris_base_with_terrain_sensors.xacro (robot description, xacro)
@@ -70,10 +70,10 @@
 		ros_topic="distance_forward"
 		min_range="0.2"
-		max_range="8.0"
+		max_range="60.0"
 		field_of_view="10"
 		ray_count="2"
 		update_rate="5"
 	>
-	  <origin xyz="0.1 0.0 -0.05" rpy="0 1.04 3.14" />
+	  <origin xyz="0.2 0.0 -0.05" rpy="0 1.05 3.14" />
 	</xacro:sonar_sensor>
 	<xacro:sonar_sensor
@@ -82,5 +82,5 @@
 		ros_topic="distance_middle"
 		min_range="0.2"
-		max_range="8.0"
+		max_range="60.0"
 		field_of_view="10"
 		ray_count="2"
@@ -94,11 +94,12 @@
 		ros_topic="distance_backward"
 		min_range="0.2"
-		max_range="8.0"
+		max_range="60.0"
 		field_of_view="10"
 		ray_count="2"
 		update_rate="5"
 	>
-	  <origin xyz="-0.1 0.0 -0.05" rpy="0 -1.04 3.14" />
+	  <origin xyz="-0.2 0.0 -0.05" rpy="0.0 1.05 0.0" />
 	</xacro:sonar_sensor>
+<!---->
 	<!-- Mount a Camera -->
 	<!--

File: models/rotors_description/urdf/with_terrain_sensors/iris_with_terrain_sensors.xacro (robot description, xacro)
@@ -9,5 +9,5 @@
   <xacro:property name="mass" value="1.5" /> <!-- [kg] -->
   <xacro:property name="body_width" value="0.47" /> <!-- [m] -->
-  <xacro:property name="body_height" value="0.11" /> <!-- [m] -->
+  <xacro:property name="body_height" value="0.05" /> <!-- [m] -->
   <xacro:property name="mass_rotor" value="0.005" /> <!-- [kg] -->
   <xacro:property name="arm_length_front_x" value="0.13" /> <!-- [m] -->
