Commit message: tilting rotors test

File: models/rotors_description/urdf/iris.xacro (robot description, xacro)
@@ -7,5 +7,5 @@
   <xacro:property name="mesh_scale" value="1 1 1"/>
   <xacro:property name="mesh_scale_prop" value="1 1 1"/>
-  <xacro:property name="mass" value="1.5" /> <!-- [kg] -->
+  <xacro:property name="mass" value="0.5" /> <!-- [kg] -->
   <xacro:property name="body_width" value="0.47" /> <!-- [m] -->
   <xacro:property name="body_height" value="0.11" /> <!-- [m] -->

File: models/rotors_description/urdf/tarot/tarot.xacro (robot description, xacro)
@@ -55,6 +55,13 @@
     <xacro:insert_block name="body_inertia" />
   </xacro:multirotor_base_macro>
+  <!--
+  <xacro:tilting_rotor
+    motor_number="0"
+    parent="base_link">
+    <origin xyz="${arm_length_front_x} -${arm_length_front_y} ${rotor_offset_top}" rpy="0 0 0" />
+  </xacro:tilting_rotor>
+  -->
   <!-- Instantiate rotors -->
-  <xacro:vertical_rotor
+  <xacro:vertical_tilting_rotor
     robot_namespace="${namespace}"
     suffix="front_right"
@@ -76,5 +83,84 @@
     <origin xyz="${arm_length_front_x} -${arm_length_front_y} ${rotor_offset_top}" rpy="0 0 0" />
     <xacro:insert_block name="rotor_inertia" />
-  </xacro:vertical_rotor>
+  </xacro:vertical_tilting_rotor>
+<xacro:vertical_tilting_rotor
+    robot_namespace="${namespace}"
+    suffix="back_left"
+    direction="ccw"
+    motor_constant="${motor_constant}"
+    moment_constant="${moment_constant}"
+    parent="base_link"
+    mass_rotor="${mass_rotor}"
+    radius_rotor="${radius_rotor}"
+    time_constant_up="${time_constant_up}"
+    time_constant_down="${time_constant_down}"
+    max_rot_velocity="${max_rot_velocity}"
+    motor_number="1"
+    rotor_drag_coefficient="${rotor_drag_coefficient}"
+    rolling_moment_coefficient="${rolling_moment_coefficient}"
+    mesh="iris_prop"
+    mesh_scale="${mesh_scale_prop}"
+    color="DarkGrey">
+    <origin xyz="-${arm_length_back_x} ${arm_length_back_y} ${rotor_offset_top}" rpy="0 0 0" />
+    <xacro:insert_block name="rotor_inertia" />
+  </xacro:vertical_tilting_rotor>
+  <xacro:vertical_tilting_rotor robot_namespace="${namespace}"
+    suffix="front_left"
+    direction="cw"
+    motor_constant="${motor_constant}"
+    moment_constant="${moment_constant}"
+    parent="base_link"
+    mass_rotor="${mass_rotor}"
+    radius_rotor="${radius_rotor}"
+    time_constant_up="${time_constant_up}"
+    time_constant_down="${time_constant_down}"
+    max_rot_velocity="${max_rot_velocity}"
+    motor_number="2"
+    rotor_drag_coefficient="${rotor_drag_coefficient}"
+    rolling_moment_coefficient="${rolling_moment_coefficient}"
+    mesh="iris_prop"
+    mesh_scale="${mesh_scale_prop}"
+    color="Blue">
+    <origin xyz="${arm_length_front_x} ${arm_length_front_y} ${rotor_offset_top}" rpy="0 0 0" />
+    <xacro:insert_block name="rotor_inertia" />
+  </xacro:vertical_tilting_rotor>
+  <xacro:vertical_tilting_rotor robot_namespace="${namespace}"
+    suffix="back_right"
+    direction="cw"
+    motor_constant="${motor_constant}"
+    moment_constant="${moment_constant}"
+    parent="base_link"
+    mass_rotor="${mass_rotor}"
+    radius_rotor="${radius_rotor}"
+    time_constant_up="${time_constant_up}"
+    time_constant_down="${time_constant_down}"
+    max_rot_velocity="${max_rot_velocity}"
+    motor_number="3"
+    rotor_drag_coefficient="${rotor_drag_coefficient}"
+    rolling_moment_coefficient="${rolling_moment_coefficient}"
+    mesh="iris_prop"
+    mesh_scale="${mesh_scale_prop}"
+    color="DarkGrey">
+    <origin xyz="-${arm_length_back_x} -${arm_length_back_y} ${rotor_offset_top}" rpy="0 0 0" />
+    <xacro:insert_block name="rotor_inertia" />
+  </xacro:vertical_tilting_rotor>
+  <!--
+  <xacro:tilting_rotor
+    motor_number="1"
+    parent="base_link">
+    <origin xyz="-${arm_length_back_x} ${arm_length_back_y} ${rotor_offset_top}" rpy="0 0 0" />
+  </xacro:tilting_rotor>
+  <xacro:tilting_rotor
+    motor_number="2"
+    parent="base_link">
+    <origin xyz="${arm_length_front_x} ${arm_length_front_y} ${rotor_offset_top}" rpy="0 0 0" />
+  </xacro:tilting_rotor>
+  <xacro:tilting_rotor
+    motor_number="3"
+    parent="base_link">
+    <origin xyz="-${arm_length_back_x} -${arm_length_back_y} ${rotor_offset_top}" rpy="0 0 0" />
+  </xacro:tilting_rotor>
+  -->
+	<!--
   <xacro:vertical_rotor
     robot_namespace="${namespace}"
@@ -138,3 +224,4 @@
     <xacro:insert_block name="rotor_inertia" />
   </xacro:vertical_rotor>
+  -->
 </robot>

File: models/rotors_description/urdf/tarot/tarot_base.xacro (robot description, xacro)
@@ -23,4 +23,5 @@
   <xacro:arg name='enable_logging' default='false' />
   <xacro:arg name='log_file' default='iris' />
+  <xacro:arg name="rotors_description_dir" default="/home/jcacace/dev/ROS/src/UAV/Firmware/Tools/sitl_gazebo/models/rotors_description"/>
   <!-- macros for gazebo plugins, sensors -->
   <xacro:include filename="$(arg rotors_description_dir)/urdf/component_snippets.xacro" />
@@ -251,3 +252,9 @@
     </xacro:bag_plugin_macro>
   </xacro:if>
+  <gazebo>
+    <plugin name="gazebo_ros_control" filename="libgazebo_ros_control.so">
+      <robotNamespace>tilt</robotNamespace>
+      <legacyModeNS>true</legacyModeNS>
+    </plugin>
+  </gazebo>
 </robot>

File: models/rotors_description/urdf/tarot_multirotor_base.xacro (robot description, xacro)
@@ -18,4 +18,16 @@
 <robot xmlns:xacro="http://ros.org/wiki/xacro">
   <!-- Main multirotor link -->
+      <xacro:macro name="transmission_block" params="joint_name">
+      <transmission name="tran1">
+        <type>transmission_interface/SimpleTransmission</type>
+          <joint name="${joint_name}">
+            <hardwareInterface>hardware_interface/PositionJointInterface</hardwareInterface>
+          </joint>
+          <actuator name="motor1">
+            <hardwareInterface>hardware_interface/PositionJointInterface</hardwareInterface>
+            <mechanicalReduction>1</mechanicalReduction>
+          </actuator>
+      </transmission>
+    </xacro:macro>
   <xacro:macro name="multirotor_base_macro"
     params="robot_namespace mass body_width body_height mesh_file mesh_scale color *inertia">
@@ -74,4 +86,40 @@
    </gazebo>
   </xacro:macro>
+	<xacro:macro name="tilting_rotor" params="motor_number parent *origin">
+		<joint name="tilt_${motor_number}_joint" type="revolute">
+			<xacro:insert_block name="origin" />
+			<axis xyz="1 0 0" />
+			<parent link="${parent}" />
+			<child link="tilt_rotor_${motor_number}" />
+			<limit lower="-1.5707963267949" upper="1.5707963267949" effort="100" velocity="1.57" />
+    </joint>
+		<link name="tilt_rotor_${motor_number}">
+		  <inertial>
+		    <origin
+		      xyz="0.0 0.0 0.0"
+		      rpy="0 0 0" />
+		    <mass
+		      value="0.01" />
+		    <inertia
+		      ixx="0"
+		      ixy="0"
+		      ixz="0"
+		      iyy="0"
+		      iyz="0"
+		      izz="0" />
+		  </inertial>
+			<visual>
+					<geometry>
+				  	<cylinder length="0.1" radius="0.01"/>
+					</geometry>
+			</visual>
+			<collision>
+				<geometry>
+					<cylinder length="0.03" radius="0.01"/>
+				</geometry>
+			</collision>
+		</link>
+    <xacro:transmission_block joint_name="tilt_${motor_number}_joint"/>
+	</xacro:macro>
   <!-- Rotor joint and link -->
   <xacro:macro name="vertical_rotor"
@@ -125,15 +173,4 @@
         <motorSpeedPubTopic>/motor_speed/${motor_number}</motorSpeedPubTopic>
         <rotorVelocitySlowdownSim>${rotor_velocity_slowdown_sim}</rotorVelocitySlowdownSim>
-        <!--
-        <gazebo_joint_control_pid>
-          <p>0.1</p>
-          <i>0</i>
-          <d>0</d>
-          <iMax>0</iMax>
-          <iMin>0</iMin>
-          <cmdMax>3</cmdMax>
-          <cmdMin>-3</cmdMin>
-        </gazebo_joint_control_pid>
-      -->
       </plugin>
     </gazebo>
@@ -142,3 +179,94 @@
     </gazebo>
   </xacro:macro>
+   <!-- Rotor joint and link -->
+  <xacro:macro name="vertical_tilting_rotor"
+    params="robot_namespace suffix direction motor_constant moment_constant parent mass_rotor radius_rotor time_constant_up time_constant_down max_rot_velocity motor_number rotor_drag_coefficient rolling_moment_coefficient color mesh mesh_scale *origin *inertia">
+    <joint name="tilt_rotor_${motor_number}_joint" type="revolute">
+      <xacro:insert_block name="origin" />
+      <axis xyz="1 0 0" />
+      <parent link="${parent}" />
+      <child link="tilt_rotor_${motor_number}" />
+      <limit lower="-1.5707963267949" upper="1.5707963267949" effort="100" velocity="1.57" />
+    </joint>
+    <link name="tilt_rotor_${motor_number}">
+		  <inertial>
+		    <origin xyz="0.0 0.0 0.0" rpy="0 0 0" />
+		    <mass value="0.01" />
+		    <inertia
+		      ixx="0"
+		      ixy="0"
+		      ixz="0"
+		      iyy="0"
+		      iyz="0"
+		      izz="0" />
+		  </inertial>
+			<visual>
+					<geometry>
+				  	<cylinder length="0.1" radius="0.01"/>
+					</geometry>
+			</visual>
+			<collision>
+				<geometry>
+					<cylinder length="0.03" radius="0.01"/>
+				</geometry>
+			</collision>
+    </link>
+    <xacro:transmission_block joint_name="tilt_rotor_${motor_number}_joint"/>
+    <joint name="rotor_${motor_number}_joint" type="continuous">
+			<origin
+      xyz="0 0.0 1.2"
+      rpy="0.0 0.0 0.0"
+			/>
+      <axis xyz="0 0 1" />
+      <!-- TODO(ff): not currently set because it's not yet supported -->
+      <!-- <limit effort="2000" velocity="${max_rot_velocity}" /> -->
+      <parent link="tilt_rotor_${motor_number}" />
+      <child link="rotor_${motor_number}" />
+    </joint>
+    <!-- TODO(ff): not currently set because it's not yet supported -->
+    <!-- <gazebo reference="rotor_${motor_number}_joint"> <axis> <xyz>0 0 1</xyz>
+      <limit> <velocity> ${max_rot_velocity} </velocity> </limit> </axis> </gazebo> -->
+    <link name="rotor_${motor_number}">
+      <inertial>
+        <mass value="${mass_rotor}" /> <!-- [kg] -->
+        <xacro:insert_block name="inertia" />
+      </inertial>
+      <visual>
+        <geometry>
+          <!-- <cylinder length="0.005" radius="${radius_rotor}"/> --> <!-- [m] -->
+          <!-- <mesh filename="package://rotors_description/meshes/propeller_${direction}.dae" -->
+          <mesh filename="package://rotors_description/meshes/${mesh}_${direction}.dae"
+            scale="${mesh_scale}" />
+          <!-- <box size="${2*radius_rotor} 0.01 0.005"/> -->
+        </geometry>
+      </visual>
+      <collision>
+        <geometry>
+          <cylinder length="0.005" radius="${radius_rotor}" /> <!-- [m] -->
+        </geometry>
+      </collision>
+    </link>
+    <gazebo>
+      <plugin name="${suffix}_motor_model" filename="libgazebo_motor_model.so">
+        <robotNamespace>${robot_namespace}</robotNamespace>
+        <jointName>rotor_${motor_number}_joint</jointName>
+        <linkName>rotor_${motor_number}</linkName>
+        <turningDirection>${direction}</turningDirection>
+        <timeConstantUp>${time_constant_up}</timeConstantUp>
+        <timeConstantDown>${time_constant_down}</timeConstantDown>
+        <maxRotVelocity>${max_rot_velocity}</maxRotVelocity>
+        <motorConstant>${motor_constant}</motorConstant>
+        <momentConstant>${moment_constant}</momentConstant>
+        <commandSubTopic>/gazebo/command/motor_speed</commandSubTopic>
+        <motorNumber>${motor_number}</motorNumber>
+        <rotorDragCoefficient>${rotor_drag_coefficient}</rotorDragCoefficient>
+        <rollingMomentCoefficient>${rolling_moment_coefficient}</rollingMomentCoefficient>
+        <motorSpeedPubTopic>/motor_speed/${motor_number}</motorSpeedPubTopic>
+        <rotorVelocitySlowdownSim>${rotor_velocity_slowdown_sim}</rotorVelocitySlowdownSim>
+      </plugin>
+    </gazebo>
+    <gazebo reference="rotor_${motor_number}">
+      <material>Gazebo/${color}</material>
+    </gazebo>
+  </xacro:macro>
 </robot>

File: models/rotors_description/urdf/tarot_with_snake/tarot_base.urdf (robot description, URDF)
Before this commit: robot iris, 31 links, 30 joints
Links:
- added link tilt_rotor_0
Joints:
- added joint tilt_rotor_0_joint: type revolute, parent base_link, child tilt_rotor_0, origin xyz=0.21 -0.21 0.033 rpy=0 0 0, axis 1 0 0, limit lower=-1.5707963267949 upper=1.5707963267949 effort=100 velocity=1.57
