Commit message: laser scanner tested

File: models/rotors_description/urdf/component_snippets.xacro (robot description, xacro)
@@ -712,4 +712,5 @@
     </joint>
     <link name="${name}_frame">
+			<!--
       <inertial>
         <mass value="0.270" />
@@ -717,4 +718,5 @@
         <inertia ixx="2.632e-4" ixy="0" ixz="0" iyy="2.632e-4" iyz="0" izz="1.62e-4" />
       </inertial>
+			-->
       <visual>
         <origin xyz="0 0 0" rpy="0 0 0" />
@@ -729,4 +731,5 @@
       </geometry>
       </collision>
+			<!---->
     </link>
   </xacro:macro>

File: models/rotors_description/urdf/with_camera/iris_base_with_camera.xacro (robot description, xacro)
@@ -90,9 +90,7 @@
 	</xacro:xtion_pro_live>
 -->
-<!--
-	    <xacro:hokuyo_utm30lx name="laser_scanner" parent="base_link" ros_topic="scan" update_rate="40" ray_count="1081" min_angle="-135" max_angle="135">
-      <origin xyz="0.3 0.2 0.06" rpy="${M_PI} 0 0"/>
-    </xacro:hokuyo_utm30lx>
-	-->
+  <xacro:hokuyo_utm30lx name="laser_scanner" parent="base_link" ros_topic="scan" update_rate="40" ray_count="1081" min_angle="-135" max_angle="135">
+    <origin xyz="0.3 0.2 0.06" rpy="${M_PI} 0 0"/>
+  </xacro:hokuyo_utm30lx>
   <!-- Mount an ADIS16448 IMU. -->
   <xacro:imu_plugin_macro

Commit message: camera and multiple sensors model

File: models/rotors_description/urdf/component_snippets.xacro (robot description, xacro)
@@ -137,4 +137,5 @@
     </joint>
     <link name="${name}_link">
+			<!--
       <inertial>
         <mass value="0.001" />
@@ -142,4 +143,5 @@
         <inertia ixx="0.000000017" ixy="0" ixz="0" iyy="0.000000017" iyz="0" izz="0.000000017" />
       </inertial>
+			-->
       <visual>
         <origin xyz="0 0 0" rpy="0 0 0" />
@@ -148,4 +150,5 @@
         </geometry>
       </visual>
+			<!--
       <collision>
         <origin xyz="0 0 0" rpy="0 0 0" />
@@ -154,4 +157,5 @@
         </geometry>
       </collision>
+			-->
     </link>
     <gazebo reference="${name}_link">
@@ -725,4 +729,5 @@
         </geometry>
       </visual>
+			<!--
       <collision>
         <origin xyz="0 0 0" rpy="0 0 0" />
@@ -731,5 +736,5 @@
       </geometry>
       </collision>
-			<!---->
+			-->
     </link>
   </xacro:macro>
@@ -851,4 +856,5 @@
     </joint>
     <link name="${name}">
+			<!--
       <inertial>
         <origin xyz="-0.00936000000 -0.00003000000 -0.00273000000" rpy="0 0 0"/>
@@ -858,4 +864,5 @@
                  izz="0.00000427339"/>
       </inertial>
+			-->
       <visual>
         <origin xyz="0 0 0" rpy="0 0 0"/>

File: models/rotors_description/urdf/with_camera/iris_base_with_camera.xacro (robot description, xacro)
@@ -65,4 +65,18 @@
   </xacro:mavlink_interface_macro>
   </xacro:if>
+	<!--
+	<xacro:sonar_sensor
+		name="sonar"
+		parent="base_link"
+		ros_topic="distance"
+		min_range="0.2"
+		max_range="8.0"
+		field_of_view="10"
+		ray_count="2"
+		update_rate="5"
+	>
+	  <origin xyz="0.0 0.0 -0.05" rpy="0 0 3.14" />
+	</xacro:sonar_sensor>
+	-->
 	<!-- Mount a Camera -->
 	<xacro:camera_macro
@@ -89,8 +103,8 @@
     <origin xyz="0 0 0" rpy="0.0 0 0.0"/>
 	</xacro:xtion_pro_live>
--->
   <xacro:hokuyo_utm30lx name="laser_scanner" parent="base_link" ros_topic="scan" update_rate="40" ray_count="1081" min_angle="-135" max_angle="135">
     <origin xyz="0.0 0.0 0.06" rpy="${M_PI} 0 0"/>
   </xacro:hokuyo_utm30lx>
+	-->
   <!-- Mount an ADIS16448 IMU. -->
   <xacro:imu_plugin_macro

File: models/rotors_description/urdf/with_sensors/iris_base_with_sensors.xacro (robot description, xacro)
@@ -65,5 +65,18 @@
   </xacro:mavlink_interface_macro>
   </xacro:if>
+	<xacro:sonar_sensor
+		name="sonar"
+		parent="base_link"
+		ros_topic="distance"
+		min_range="0.2"
+		max_range="8.0"
+		field_of_view="10"
+		ray_count="2"
+		update_rate="5"
+	>
+	  <origin xyz="0.0 0.0 -0.05" rpy="0 0 3.14" />
+	</xacro:sonar_sensor>
 	<!-- Mount a Camera -->
+	<!--
 	<xacro:camera_macro
 		  namespace="${namespace}"
@@ -84,15 +97,12 @@
 		<origin xyz="0.12 0 -0.02" rpy="0.0 1.1 0.0" />
 	</xacro:camera_macro>
-	<!--
+	-->
   <xacro:xtion_pro_live name="rgbd_camera" parent="base_link">
 	 	<origin xyz="0.11 0.0 -0.02" rpy="0.0 0.95 0.0"/>
     <origin xyz="0 0 0" rpy="0.0 0 0.0"/>
 	</xacro:xtion_pro_live>
--->
-<!--
-	    <xacro:hokuyo_utm30lx name="laser_scanner" parent="base_link" ros_topic="scan" update_rate="40" ray_count="1081" min_angle="-135" max_angle="135">
-      <origin xyz="0.3 0.2 0.06" rpy="${M_PI} 0 0"/>
-    </xacro:hokuyo_utm30lx>
-	-->
+  <xacro:hokuyo_utm30lx name="laser_scanner" parent="base_link" ros_topic="scan" update_rate="40" ray_count="1081" min_angle="-135" max_angle="135">
+    <origin xyz="0.0 0.0 0.06" rpy="${M_PI} 0 0"/>
+  </xacro:hokuyo_utm30lx>
   <!-- Mount an ADIS16448 IMU. -->
   <xacro:imu_plugin_macro
@@ -114,16 +124,4 @@
     <origin xyz="0 0 0" rpy="0 0 0" />
   </xacro:imu_plugin_macro>
-	<xacro:sonar_sensor
-		name="sonar"
-		parent="base_link"
-		ros_topic="distance"
-		min_range="0.2"
-		max_range="8.0"
-		field_of_view="10"
-		ray_count="2"
-		update_rate="5"
-	>
-	  <origin xyz="0.0 0.0 -0.04" rpy="0 0 3.14" />
-	</xacro:sonar_sensor>
   <xacro:if value="$(arg enable_ground_truth)">
     <!-- Mount an IMU providing ground truth. -->

Commit message: added uav with ARVA

File: models/rotors_description/urdf/component_snippets.xacro (robot description, xacro)
@@ -193,4 +193,50 @@
       </sensor>
     </gazebo>
+  </xacro:macro>
+  <xacro:macro name="artva_macro" params="channels frame_id *origin">
+    <link name="receiver">
+			<!--
+		  <collision>
+		    <origin xyz="-0.12 0.0 0.0" rpy="0 0 0"/>
+		    <geometry>
+		      <box size="0.05 0.05 0.05"/>
+		    </geometry>
+		  </collision>
+			-->
+		  <visual>
+		    <origin xyz="-0.18 0.0 0.0" rpy="0 0 0"/>
+		    <geometry>
+		      <box size="0.01 0.01 0.01"/>
+		    </geometry>
+		    <material name="orange"/>
+		  </visual>
+			<!--
+		  <inertial>
+		    <origin xyz="0 0 1" rpy="0 0 0"/>
+		    <mass value="1"/>
+		    <inertia
+		      ixx="1.0" ixy="0.0" ixz="0.0"
+		      iyy="1.0" iyz="0.0"
+		      izz="1.0"/>
+		  </inertial>
+			-->
+		</link>
+ 		<joint name="receiver_joint" type="fixed">
+      <xacro:insert_block name="origin" />
+      <parent link="base_link" />
+      <child link="receiver" />
+    </joint>
+		<material name="orange">
+		  <color rgba="${255/255} ${108/255} ${10/255} 1.0"/>
+		</material>
+		<gazebo reference="receiver">
+		  <material>Gazebo/Orange</material>
+		</gazebo>
+		<gazebo>
+			<plugin filename="libarva_sim_receiver.so" name="receiver">
+				<channels>${channels}</channels>
+				<frame_id>${frame_id}</frame_id>
+		  </plugin>
+		</gazebo>
   </xacro:macro>
   <!-- Macro to add the mavlink interface. -->

Commit message: Arva fsupport file added

File: models/rotors_description/urdf/component_snippets.xacro (robot description, xacro)
@@ -194,14 +194,6 @@
     </gazebo>
   </xacro:macro>
-  <xacro:macro name="artva_macro" params="channels frame_id *origin">
+  <xacro:macro name="arva_macro" params="channels frame_id sensor_name *origin">
     <link name="receiver">
-			<!--
-		  <collision>
-		    <origin xyz="-0.12 0.0 0.0" rpy="0 0 0"/>
-		    <geometry>
-		      <box size="0.05 0.05 0.05"/>
-		    </geometry>
-		  </collision>
-			-->
 		  <visual>
 		    <origin xyz="-0.18 0.0 0.0" rpy="0 0 0"/>
@@ -211,14 +203,4 @@
 		    <material name="orange"/>
 		  </visual>
-			<!--
-		  <inertial>
-		    <origin xyz="0 0 1" rpy="0 0 0"/>
-		    <mass value="1"/>
-		    <inertia
-		      ixx="1.0" ixy="0.0" ixz="0.0"
-		      iyy="1.0" iyz="0.0"
-		      izz="1.0"/>
-		  </inertial>
-			-->
 		</link>
  		<joint name="receiver_joint" type="fixed">
@@ -236,4 +218,5 @@
 			<plugin filename="libarva_sim_receiver.so" name="receiver">
 				<channels>${channels}</channels>
+				<sensor_name>${sensor_name}</sensor_name>
 				<frame_id>${frame_id}</frame_id>
 		  </plugin>

File: models/rotors_description/urdf/with_artva/iris_base_with_artva.xacro (robot description, xacro)
@@ -97,7 +97,7 @@
 		<origin xyz="0.12 0 -0.02" rpy="0.0 1.1 0.0" />
 	</xacro:camera_macro>
-	<xacro:artva_macro channels="2" frame_id="artva">
+	<xacro:arva_macro channels="1" frame_id="artva" sensor_name="receiver1">
 		      <origin xyz="0 0 0" rpy="0 0 0" />
-	</xacro:artva_macro>
+	</xacro:arva_macro>
 	<!--
   <xacro:xtion_pro_live name="rgbd_camera" parent="base_link">

Commit message: sitl standalone

File: models/rotors_description/urdf/component_snippets.xacro (robot description, xacro)
@@ -223,5 +223,5 @@
 		</gazebo>
   </xacro:macro>
-  <!-- Macro to add the mavlink interface. -->
+<!-- Macro to add the mavlink interface. -->
   <xacro:macro name="mavlink_interface_macro" params="namespace imu_sub_topic gps_sub_topic mavlink_addr mavlink_udp_port serial_enabled serial_device baudrate qgc_addr qgc_udp_port hil_mode hil_state_level vehicle_is_tailsitter send_odometry">
     <gazebo>
@@ -343,4 +343,123 @@
     </gazebo>
   </xacro:macro>
+<!-- Macro to add the mavlink interface. -->
+  <xacro:macro name="ros_interface_macro" params="namespace imu_sub_topic gps_sub_topic mavlink_addr mavlink_udp_port serial_enabled serial_device baudrate qgc_addr qgc_udp_port hil_mode hil_state_level vehicle_is_tailsitter send_odometry">
+    <gazebo>
+      <plugin name="ros_interface" filename="libgazebo_ros_interface.so">
+        <robotNamespace>${namespace}</robotNamespace>
+        <imuSubTopic>${imu_sub_topic}</imuSubTopic>
+        <gpsSubTopic>${gps_sub_topic}</gpsSubTopic>
+        <mavlink_addr>$(arg mavlink_addr)</mavlink_addr>
+        <mavlink_udp_port>$(arg mavlink_udp_port)</mavlink_udp_port>
+        <serialEnabled>$(arg serial_enabled)</serialEnabled>
+        <serialDevice>$(arg serial_device)</serialDevice>
+        <baudRate>$(arg baudrate)</baudRate>
+        <qgc_addr>$(arg qgc_addr)</qgc_addr>
+        <qgc_udp_port>$(arg qgc_udp_port)</qgc_udp_port>
+        <hil_mode>$(arg hil_mode)</hil_mode>
+        <hil_state_level>$(arg hil_state_level)</hil_state_level>
+        <vehicle_is_tailsitter>$(arg vehicle_is_tailsitter)</vehicle_is_tailsitter>
+        <send_odometry>$(arg send_odometry)</send_odometry>
+        <motorSpeedCommandPubTopic>/gazebo/command/motor_speed</motorSpeedCommandPubTopic>
+        <control_channels>
+          <channel name="rotor1">
+            <input_index>0</input_index>
+            <input_offset>0</input_offset>
+            <input_scaling>1000</input_scaling>
+            <zero_position_disarmed>0</zero_position_disarmed>
+            <zero_position_armed>100</zero_position_armed>
+            <joint_control_type>velocity</joint_control_type>
+          </channel>
+          <channel name="rotor2">
+            <input_index>1</input_index>
+            <input_offset>0</input_offset>
+            <input_scaling>1000</input_scaling>
+            <zero_position_disarmed>0</zero_position_disarmed>
+            <zero_position_armed>100</zero_position_armed>
+            <joint_control_type>velocity</joint_control_type>
+          </channel>
+          <channel name="rotor3">
+            <input_index>2</input_index>
+            <input_offset>0</input_offset>
+            <input_scaling>1000</input_scaling>
+            <zero_position_disarmed>0</zero_position_disarmed>
+            <zero_position_armed>100</zero_position_armed>
+            <joint_control_type>velocity</joint_control_type>
+          </channel>
+          <channel name="rotor4">
+            <input_index>3</input_index>
+            <input_offset>0</input_offset>
+            <input_scaling>1000</input_scaling>
+            <zero_position_disarmed>0</zero_position_disarmed>
+            <zero_position_armed>100</zero_position_armed>
+            <joint_control_type>velocity</joint_control_type>
+          </channel>
+          <channel name="rotor5">
+            <input_index>4</input_index>
+            <input_offset>1</input_offset>
+            <input_scaling>324.6</input_scaling>
+            <zero_position_disarmed>0</zero_position_disarmed>
+            <zero_position_armed>0</zero_position_armed>
+            <joint_control_type>velocity</joint_control_type>
+            <joint_control_pid>
+              <p>0.1</p>
+              <i>0</i>
+              <d>0</d>
+              <iMax>0.0</iMax>
+              <iMin>0.0</iMin>
+              <cmdMax>2</cmdMax>
+              <cmdMin>-2</cmdMin>
+            </joint_control_pid>
+            <joint_name>zephyr_delta_wing::propeller_joint</joint_name>
+          </channel>
+          <channel name="rotor6">
+            <input_index>5</input_index>
+            <input_offset>0</input_offset>
+            <input_scaling>0.524</input_scaling>
+            <zero_position_disarmed>0</zero_position_disarmed>
+            <zero_position_armed>0</zero_position_armed>
+            <joint_control_type>position</joint_control_type>
+            <joint_name>zephyr_delta_wing::flap_left_joint</joint_name>
+            <joint_control_pid>
+              <p>10.0</p>
+              <i>0</i>
+              <d>0</d>
+              <iMax>0</iMax>
+              <iMin>0</iMin>
+              <cmdMax>20</cmdMax>
+              <cmdMin>-20</cmdMin>
+            </joint_control_pid>
+          </channel>
+          <channel name="rotor7">
+            <input_index>6</input_index>
+            <input_offset>0</input_offset>
+            <input_scaling>0.524</input_scaling>
+            <zero_position_disarmed>0</zero_position_disarmed>
+            <zero_position_armed>0</zero_position_armed>
+            <joint_control_type>position</joint_control_type>
+            <joint_name>zephyr_delta_wing::flap_right_joint</joint_name>
+            <joint_control_pid>
+              <p>10.0</p>
+              <i>0</i>
+              <d>0</d>
+              <iMax>0</iMax>
+              <iMin>0</iMin>
+              <cmdMax>20</cmdMax>
+              <cmdMin>-20</cmdMin>
+            </joint_control_pid>
+          </channel>
+          <channel name="rotor8">
+            <input_index>7</input_index>
+            <input_offset>0</input_offset>
+            <input_scaling>0.524</input_scaling>
+            <zero_position_disarmed>0</zero_position_disarmed>
+            <zero_position_armed>0</zero_position_armed>
+            <joint_control_type>position</joint_control_type>
+          </channel>
+        </control_channels>
+      </plugin>
+    </gazebo>
+  </xacro:macro>
+<!---->
   <!-- Macro to add an IMU. -->
   <xacro:macro name="imu_plugin_macro"

File: models/rotors_description/urdf/tarot_standalone/tarot_base.xacro (robot description, xacro)
@@ -17,5 +17,6 @@
   <xacro:arg name='vehicle_is_tailsitter' default='false' />
   <xacro:arg name='visual_material' default='DarkGrey' />
-  <xacro:arg name='enable_mavlink_interface' default='true' />
+  <xacro:arg name='enable_mavlink_interface' default='false' />
+  <xacro:arg name='enable_ros_interface' default='true' />
   <xacro:arg name='enable_wind' default='false' />
   <!-- The following causes segfault with multiple vehicles if defaults to true!!! -->
@@ -46,7 +47,5 @@
     >
   </xacro:gps_plugin_macro>
-  <xacro:if value="$(arg enable_mavlink_interface)">
-  <!-- Instantiate mavlink telemetry interface. -->
-  <xacro:mavlink_interface_macro
+  <xacro:ros_interface_macro
     namespace="${namespace}"
     imu_sub_topic="/imu"
@@ -64,114 +63,6 @@
     send_odometry="$(arg send_odometry)"
     >
-  </xacro:mavlink_interface_macro>
-  </xacro:if>
-	<!-- Mount a Camera
-	<xacro:camera_macro
-		  namespace="${namespace}"
-			parent_link="base_link"
-			camera_suffix="raw"
-			frame_rate="30"
-			horizontal_fov="1.4"
-			image_width="1280"
-			image_height="720"
-			image_format="B8G8R8"
-			min_distance="0.02"
-			max_distance="300"
-			noise_mean="0.0"
-			noise_stddev="0.008"
-			enable_visual="1"
-		>
-		<box size="0.02 0.02 0.02" />
-		<origin xyz="0.12 0 -0.02" rpy="0.0 1.1 0.0" />
-	</xacro:camera_macro>
--->
-	<!--
-  <xacro:xtion_pro_live name="rgbd_camera" parent="base_link">
-	 	<origin xyz="0.11 0.0 -0.02" rpy="0.0 0.95 0.0"/>
-    <origin xyz="0 0 0" rpy="0.0 0 0.0"/>
-	</xacro:xtion_pro_live>
-	    <xacro:hokuyo_utm30lx name="laser_scanner" parent="base_link" ros_topic="scan" update_rate="40" ray_count="1081" min_angle="-135" max_angle="135">
-      <origin xyz="0.0 0.0 0.06" rpy="${M_PI} 0 0"/>
-    </xacro:hokuyo_utm30lx>
--->
-	<!--
-	<xacro:macro name="hokuyo_utm30lx_model" params="name parent *origin">
-    <joint name="${name}_joint" type="fixed">
-      <xacro:insert_block name="origin" />
-      <parent link="${parent}"/>
-      <child link="${name}_frame"/>
-    </joint>
-    <link name="${name}_frame">
-      <inertial>
-        <mass value="0.270" />
-        <origin xyz="0 0 0" rpy="0 0 0" />
-        <inertia ixx="2.632e-4" ixy="0" ixz="0" iyy="2.632e-4" iyz="0" izz="1.62e-4" />
-      </inertial>
-      <visual>
-        <origin xyz="0 0 0" rpy="0 0 0" />
-        <geometry>
-        <box size="0.025 0.025 0.035" />
-        </geometry>
-      </visual>
-      <collision>
-        <origin xyz="0 0 0" rpy="0 0 0" />
-        <geometry>
-        <box size="0.025 0.025 0.035" />
-      </geometry>
-      </collision>
-    </link>
-  </xacro:macro>
-	<xacro:macro name="hokuyo_utm30lx" params="name parent *origin ros_topic update_rate ray_count min_angle max_angle">
-      <xacro:hokuyo_utm30lx_model name="${name}" parent="${parent}">
-        <xacro:insert_block name="origin" />
-      </xacro:hokuyo_utm30lx_model>
-      <gazebo reference="${name}_frame">
-        <sensor type="ray" name="${name}">
-          <always_on>true</always_on>
-          <update_rate>${update_rate}</update_rate>
-          <pose>0 0 0.0 0 0 0</pose>
-          <visualize>false</visualize>
-          <ray>
-            <scan>
-              <horizontal>
-                <samples>${ray_count}</samples>
-                <resolution>1</resolution>
-                <min_angle>${min_angle * M_PI/180}</min_angle>
-                <max_angle>${max_angle * M_PI/180}</max_angle>
-              </horizontal>
-            </scan>
-            <range>
-              <min>0.2</min>
-              <max>30.0</max>
-              <resolution>0.01</resolution>
-            </range>
-            <noise>
-              <type>gaussian</type>
-              <mean>0.0</mean>
-              <stddev>0.004</stddev>
-            </noise>
-          </ray>
-          <plugin name="gazebo_ros_${name}_controller" filename="libgazebo_ros_laser.so">
-            <topicName>${ros_topic}</topicName>
-            <frameName>${name}_frame</frameName>
-          </plugin>
-        </sensor>
-      </gazebo>
-   </xacro:macro>
-	-->
-	<!--
-	<xacro:sonar_sensor
-		name="sonar"
-		parent="base_link"
-		ros_topic="sonar"
-		min_range="0.2"
-		max_range="8.0"
-		field_of_view="10"
-		ray_count="2"
-		update_rate="5"
-	>
-  <origin xyz="0.0 0.0 -0.04" rpy="0 0 3.14" />
-	</xacro:sonar_sensor>
-	-->
+  </xacro:ros_interface_macro>
+<!---->
   <xacro:hokuyo_utm30lx name="laser_scanner" parent="base_link" ros_topic="scan" update_rate="40" ray_count="1081" min_angle="-135" max_angle="135">
     <origin xyz="0.0 0.0 0.1" rpy="${M_PI} 0 0"/>
