Commit message: tarot with tilting rotors

File: models/rotors_description/urdf/tarot/tarot_base.xacro (robot description, xacro)
@@ -23,5 +23,5 @@
   <xacro:arg name='enable_logging' default='false' />
   <xacro:arg name='log_file' default='iris' />
-  <xacro:arg name="rotors_description_dir" default="/home/jcacace/dev/ROS/src/UAV/Firmware/Tools/sitl_gazebo/models/rotors_description"/>
+  <xacro:arg name="rotors_description_dir" default="/home/jcacace/dev/ros_ws/src/Firmware/Tools/sitl_gazebo/models/rotors_description"/>
   <!-- macros for gazebo plugins, sensors -->
   <xacro:include filename="$(arg rotors_description_dir)/urdf/component_snippets.xacro" />

File: models/rotors_description/urdf/tarot_multirotor_base.xacro (robot description, xacro)
@@ -182,4 +182,5 @@
   <xacro:macro name="vertical_tilting_rotor"
     params="robot_namespace suffix direction motor_constant moment_constant parent mass_rotor radius_rotor time_constant_up time_constant_down max_rot_velocity motor_number rotor_drag_coefficient rolling_moment_coefficient color mesh mesh_scale *origin *inertia">
+		<!-- -->
     <joint name="tilt_rotor_${motor_number}_joint" type="revolute">
       <xacro:insert_block name="origin" />
@@ -192,34 +193,42 @@
 		  <inertial>
 		    <origin xyz="0.0 0.0 0.0" rpy="0 0 0" />
-		    <mass value="0.01" />
+		    <mass value="0.1" />
 		    <inertia
-		      ixx="0"
+		      ixx="0.001"
 		      ixy="0"
 		      ixz="0"
-		      iyy="0"
+		      iyy="0.001"
 		      iyz="0"
-		      izz="0" />
+		      izz="0.001" />
 		  </inertial>
 			<visual>
 					<geometry>
-				  	<cylinder length="0.1" radius="0.01"/>
+				  	<cylinder length="0.02" radius="0.01"/>
 					</geometry>
 			</visual>
 			<collision>
 				<geometry>
-					<cylinder length="0.03" radius="0.01"/>
+					<cylinder length="0.02" radius="0.01"/>
 				</geometry>
 			</collision>
     </link>
     <xacro:transmission_block joint_name="tilt_rotor_${motor_number}_joint"/>
+		<!-- -->
     <joint name="rotor_${motor_number}_joint" type="continuous">
+			<!---->
 			<origin
-      xyz="0 0.0 1.2"
+      xyz="0 0.0 0.018"
       rpy="0.0 0.0 0.0"
 			/>
+			<!--
+			<xacro:insert_block name="origin" />
+      -->
       <axis xyz="0 0 1" />
       <!-- TODO(ff): not currently set because it's not yet supported -->
       <!-- <limit effort="2000" velocity="${max_rot_velocity}" /> -->
-      <parent link="tilt_rotor_${motor_number}" />
+			<parent link="tilt_rotor_${motor_number}" />
+      <!--
+			<parent link="${parent}" />
+			-->
       <child link="rotor_${motor_number}" />
     </joint>

Commit message: tarot tilting and with sensors

File: models/rotors_description/urdf/tarot/tarot_base.xacro (robot description, xacro)
@@ -23,5 +23,5 @@
   <xacro:arg name='enable_logging' default='false' />
   <xacro:arg name='log_file' default='iris' />
-  <xacro:arg name="rotors_description_dir" default="/home/jcacace/dev/ros_ws/src/Firmware/Tools/sitl_gazebo/models/rotors_description"/>
+  <xacro:arg name="rotors_description_dir" default="/home/jcacace/dev/ROS/src/UAV/Firmware/Tools/sitl_gazebo/models/rotors_description"/>
   <!-- macros for gazebo plugins, sensors -->
   <xacro:include filename="$(arg rotors_description_dir)/urdf/component_snippets.xacro" />
@@ -173,4 +173,11 @@
 	</xacro:sonar_sensor>
 	-->
+  <xacro:hokuyo_utm30lx name="laser_scanner" parent="base_link" ros_topic="scan" update_rate="40" ray_count="1081" min_angle="-135" max_angle="135">
+    <origin xyz="0.0 0.0 0.06" rpy="${M_PI} 0 0"/>
+  </xacro:hokuyo_utm30lx>
+  <xacro:xtion_pro_live name="rgbd_camera" parent="base_link">
+	 	<origin xyz="0.11 0.0 -0.02" rpy="0.0 0.95 0.0"/>
+    <origin xyz="0 0 0" rpy="0.0 0 0.0"/>
+	</xacro:xtion_pro_live>
   <!-- Mount an ADIS16448 IMU. -->
   <xacro:imu_plugin_macro

File: models/rotors_description/urdf/tarot_with_snake/tarot_base.urdf (robot description, URDF)
Before this commit: robot iris, 32 links, 31 joints
Links:
- added link tilt_rotor_1, mass 0.1; collision cylinder length=0.02 radius=0.01; visual cylinder length=0.02 radius=0.01
- added link tilt_rotor_2, mass 0.1; collision cylinder length=0.02 radius=0.01; visual cylinder length=0.02 radius=0.01
- added link tilt_rotor_3, mass 0.1; collision cylinder length=0.02 radius=0.01; visual cylinder length=0.02 radius=0.01
- link tilt_rotor_0: mass None -> 0.1; geometry collision cylinder length=0.02 radius=0.01; visual cylinder length=0.02 radius=0.01
Joints:
- added joint tilt_rotor_1_joint: type revolute, parent base_link, child tilt_rotor_1, origin xyz=-0.21 0.21 0.033 rpy=0 0 0, axis 1 0 0, limit lower=-1.5707963267949 upper=1.5707963267949 effort=100 velocity=1.57
- added joint tilt_rotor_2_joint: type revolute, parent base_link, child tilt_rotor_2, origin xyz=0.21 0.21 0.033 rpy=0 0 0, axis 1 0 0, limit lower=-1.5707963267949 upper=1.5707963267949 effort=100 velocity=1.57
- added joint tilt_rotor_3_joint: type revolute, parent base_link, child tilt_rotor_3, origin xyz=-0.21 -0.21 0.033 rpy=0 0 0, axis 1 0 0, limit lower=-1.5707963267949 upper=1.5707963267949 effort=100 velocity=1.57
- joint rotor_0_joint: origin xyz=0.21 -0.21 0.033 rpy=0 0 0 -> xyz=0 0.0 0.018 rpy=0.0 0.0 0.0; parent base_link -> tilt_rotor_0
- joint rotor_1_joint: origin xyz=-0.21 0.21 0.033 rpy=0 0 0 -> xyz=0 0.0 0.018 rpy=0.0 0.0 0.0; parent base_link -> tilt_rotor_1
- joint rotor_2_joint: origin xyz=0.21 0.21 0.033 rpy=0 0 0 -> xyz=0 0.0 0.018 rpy=0.0 0.0 0.0; parent base_link -> tilt_rotor_2
- joint rotor_3_joint: origin xyz=-0.21 -0.21 0.033 rpy=0 0 0 -> xyz=0 0.0 0.018 rpy=0.0 0.0 0.0; parent base_link -> tilt_rotor_3
